File: docs/Eagle/CurrentMeter2.sch (EAGLE design)
At the start: 4 parts

Commit message: schematics finalized
Connections:
- net N$5 renamed 3.3V
Other:
- note added: "AC/DC Adapter 5V"
- note added: "Dryer"
- note added: "Washer"
- note added: "YHDC SC Transformer Dryer"
- note added: "YHDC SC Transformer Washer"
- note removed: "AC/DC"
- note removed: "GND"
Changed lines of the file:
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@@
 <part name="SOCKET1" library="con-avx" library_urn="urn:adsk.eagle:library:129" deviceset="009175003" device="" package3d_urn="urn:adsk.eagle:package:6128/1" value=""/>
 <part name="SOCKET2" library="con-avx" library_urn="urn:adsk.eagle:library:129" deviceset="009175003" device="" package3d_urn="urn:adsk.eagle:package:6128/1" value=""/>
+<part name="GND" library="SparkFun-PowerSymbols" library_urn="urn:adsk.eagle:library:530" deviceset="GND2" device="" value="GND"/>
 </parts>
 <sheets>
@@
 <text x="-20.32" y="-5.08" size="1.778" layer="91">L</text>
 <text x="50.8" y="-5.08" size="1.778" layer="91">N</text>
-<text x="38.1" y="-5.08" size="1.778" layer="91">GND</text>
-<text x="9.398" y="26.162" size="1.778" layer="91">AC/DC</text>
+<text x="8.636" y="19.812" size="1.778" layer="91">AC/DC
+Adapter
+5V</text>
+<text x="10.16" y="76.2" size="1.778" layer="91">YHDC SC
+Transformer
+Washer</text>
+<text x="10.16" y="48.26" size="1.778" layer="91">YHDC SC
+Transformer
+Dryer</text>
+<text x="27.94" y="91.44" size="1.778" layer="91">Washer</text>
+<text x="27.94" y="63.5" size="1.778" layer="91">Dryer</text>
 </plain>
 <instances>
@@
 <attribute name="NAME" x="25.4" y="68.58" size="1.778" layer="95" rot="R270"/>
 <attribute name="VALUE" x="36.83" y="58.42" size="1.778" layer="96" rot="R90"/>
+</instance>
+<instance part="GND" gate="G$1" x="40.64" y="-2.54" smashed="yes">
+<attribute name="VALUE" x="40.64" y="-4.318" size="1.778" layer="96" align="top-center"/>
 </instance>
 </instances>
@@
 </segment>
 </net>
-<net name="N$5" class="0">
+<net name="3.3V" class="0">
 <segment>
-<wire x1="40.64" y1="-2.54" x2="40.64" y2="45.72" width="0.1524" layer="91"/>
+<wire x1="40.64" y1="-2.54" x2="40.64" y2="0" width="0.1524" layer="91"/>
+<wire x1="40.64" y1="0" x2="40.64" y2="45.72" width="0.1524" layer="91"/>
 <wire x1="40.64" y1="45.72" x2="30.48" y2="45.72" width="0.1524" layer="91"/>
 <pinref part="SOCKET2" gate="G$1" pin="2@1"/>
@@
 <pinref part="SOCKET1" gate="G$1" pin="2@1"/>
 <wire x1="30.48" y1="73.66" x2="30.48" y2="81.28" width="0.1524" layer="91"/>
+<pinref part="GND" gate="G$1" pin="3.3V"/>
+<junction x="40.64" y="0"/>
 </segment>
 </net>
@@
 </drawing>
 <compatibility>
+<note version="6.3" minversion="6.2.2" severity="warning">
+Since Version 6.2.2 text objects can contain more than one line,
+which will not be processed correctly with this version.
+</note>
 <note version="8.2" severity="warning">
 Since Version 8.2, EAGLE supports online libraries. The ids
