File: docs/Eagle/InfoDashboard.sch (EAGLE design)
At the start: 3 parts, among them X1 HD44780LCD-1602

Commit message: documentation
Parts:
- added IC1: (no value), DC_LOAD_AU:78LXX
- added R1: (no value), eagle-ltspice:R
Changed lines of the file:
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@@
 <?xml version="1.0" encoding="utf-8"?>
 <!DOCTYPE eagle SYSTEM "eagle.dtd">
-<eagle version="9.4.1">
+<eagle version="9.4.2">
 <drawing>
 <settings>
@@
 <part name="U1" library="esp8266modules" deviceset="ESP12" device=""/>
 <part name="X1" library="adafruit" library_urn="urn:adsk.eagle:library:420" deviceset="HD44780LCD" device="-1602" package3d_urn="urn:adsk.eagle:package:6240760/1"/>
+<part name="IC1" library="DC_LOAD_AU" library_urn="urn:adsk.eagle:library:220454" deviceset="78LXX" device="" package3d_urn="urn:adsk.eagle:package:220577/2"/>
+<part name="R1" library="eagle-ltspice" library_urn="urn:adsk.eagle:library:217" deviceset="R" device="" package3d_urn="urn:adsk.eagle:package:13300/1"/>
 </parts>
 <sheets>
@@
 <attribute name="VALUE" x="114.3" y="-5.08" size="2.1844" layer="96" font="vector"/>
 </instance>
+<instance part="IC1" gate="1" x="76.2" y="12.7" smashed="yes">
+<attribute name="NAME" x="78.74" y="5.08" size="1.778" layer="95"/>
+<attribute name="VALUE" x="78.74" y="2.54" size="1.778" layer="96"/>
+</instance>
+<instance part="R1" gate="G$1" x="53.34" y="5.08" smashed="yes">
+<attribute name="NAME" x="49.53" y="6.5786" size="1.778" layer="95"/>
+<attribute name="VALUE" x="49.53" y="1.778" size="1.778" layer="96"/>
+</instance>
 </instances>

Commit message: schematics finalized
Parts:
- removed IC1: (no value), DC_LOAD_AU:78LXX
- removed R1: (no value), eagle-ltspice:R
- removed X1: HD44780LCD-1602, adafruit:HD44780LCD-1602
- added CAPACITOR: 10 mF, Nordic_nRF:CAPACITOR_0201_L
- added CAPACITOR1: 100 nF, Nordic_nRF:CAPACITOR_0201_L
- added RESISTOR: 2K Ohm, eagle-ltspice:R
- added U$3: LCD 20x4, HD44780LCD2:LCD-HD4478016X2-4-HOLES-BL16X2-4-HOLES-BL
- added U$4: LCD-I2C-CONVERTER, diy-modules:LCD-I2C-CONVERTER
- added VREGULATOR: 3.3V, DC_LOAD_AU:78LXX
- B1: value ARDUINO_UNO_R3 -> ARDUINO_NANO
- ESP8266: value (none) -> ESP12
- renumbered U1 to ESP8266
Connections:
- new net N$1: B1.*D9, ESP8266.TX
- new net N$10: U$3.DB2, U$4.DB2
- new net N$11: U$3.DB3, U$4.DB3
- new net N$12: U$3.DB4, U$4.DB4
- new net N$13: U$3.DB5, U$4.DB5
- new net N$14: U$3.DB6, U$4.DB6
- new net N$15: U$3.DB7, U$4.DB7
- new net N$16: U$3.A, U$4.LED.A
- new net N$17: U$3.K, U$4.LED.K
- new net N$18: B1.A4, U$4.SDA
- new net N$19: B1.GND, CAPACITOR.2, CAPACITOR1.2, ESP8266.GND, ESP8266.GPIO15, U$4.GND, VREGULATOR.GND
- new net N$2: U$3.VSS, U$4.VSS
- new net N$20: B1.D8, B1.VCC, CAPACITOR1.1, ESP8266.RX, U$4.VCC, VREGULATOR.IN
- new net N$21: CAPACITOR.1, ESP8266.CH_PD, ESP8266.VCC, VREGULATOR.OUT
- new net N$22: B1.A5, U$4.SCL
- new net N$23: RESISTOR.1
- new net N$24: RESISTOR.2
- new net N$3: U$3.VDD, U$4.VDD
- new net N$4: U$3.VO, U$4.VEE
- new net N$5: U$3.RS, U$4.RS
- new net N$6: U$3.R/W, U$4.R/W
- new net N$7: U$3.E, U$4.EN
- new net N$8: U$3.DB0, U$4.DB0
- new net N$9: U$3.DB1, U$4.DB1
Other:
- note added: "5V DC"
- note added: "GND"
- moved on the sheet: B1
